Commit message: Add fixed joint between base_link and chassis_1 in SMART-TROLLEY V5 model

File: description/SMART-TROLLEY_V5.xacro (robot description, xacro)
@@ -84,4 +84,9 @@
   </collision>
 </link>
+<joint name="base_to_chassis" type="fixed">
+  <origin xyz="0 0 0" rpy="0 0 0"/>
+  <parent link="base_link"/>
+  <child link="chassis_1"/>
+</joint>
 <joint name="left_wheel_joint" type="continuous">
   <origin xyz="-0.099914 0.000901 0.335814" rpy="0 0 0"/>
